File: Schematic_PCB/Radio2.kicad_pcb (KiCad board)
At the start: 2 copper layers, 66.5 x 109.8 mm, 17 parts, among them J1 Conn_Coaxial, SW1 SW_Push, SW2 SW_Push, SW3 SW_Push, U2 SX1272, U3 MAX98357A, U4 MCP1826S, U5 Industrial Monitor, Color LCD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, U6 ESP32-DEVKITC V4

Commit message: upload new files
Parts:
- moved J1 17.4 mm to (174.2, 56.2)
- moved BT1 5.11 mm to (118.5, 103.0), turned to -90 degrees
Routing:
- net Net-(J1-In): track 74.3 -> 85.1 mm, vias 0 -> 2
- net Net-(BT1-+): track 22.0 -> 14.3 mm
- net GND: track 176.3 -> 180.9 mm
- net Net-(U2-DIO0): track 26.9 -> 25.5 mm
- net Net-(U3-OUTP): track 9.68 -> 11.1 mm
- net Net-(U6-IO32): track 70.2 -> 69.2 mm
Other:
- board size 66.5 x 109.8 mm -> 73.2 x 98 mm
